Commit message: added links and joints fro all wheels

File: urdf/my_robot.urdf (robot description, URDF)
Before this commit: robot ASHWINI, 1 links, 0 joints
Links:
- added link base_footprint
- added link caster_wheel; visual sphere radius=0.05
- added link left_wheel; visual cylinder length=0.05 radius=0.1
- added link lidar; visual cylinder length=0.05 radius=0.1
- added link right_wheel; visual cylinder length=0.05 radius=0.1
Joints:
- added joint base_caster_wheel_joint: type fixed, parent base_link, child caster_wheel, origin xyz=0.2 0 -0.05 rpy=0 0 0, axis 0 1 0
- added joint base_joint: type fixed, parent base_footprint, child base_link, origin xyz=0 0 0.1 rpy=0 0 0
- added joint base_left_wheel_joint: type continuous, parent base_link, child left_wheel, origin xyz=-0.15 0.225 0 rpy=0 0 0, axis 0 1 0
- added joint base_lidar_joint: type fixed, parent base_link, child lidar, origin xyz=0 0 0.225 rpy=0 0 0
- added joint base_right_wheel_joint: type continuous, parent base_link, child right_wheel, origin xyz=-0.15 -0.225 0 rpy=0 0 0, axis 0 1 0

Commit message: added intertial tags, teleop key

File: urdf/my_robot.urdf (robot description, URDF)
Before this commit: robot ASHWINI, 6 links, 5 joints
Links:
- link base_link: mass None -> 5.0; geometry collision box size=0.6 0.4 0.2; visual box size=0.6 0.4 0.2
- link caster_wheel: mass None -> 0.2; geometry collision sphere radius=0.05; visual sphere radius=0.05
- link left_wheel: mass None -> 0.5; geometry collision cylinder length=0.05 radius=0.1; visual cylinder length=0.05 radius=0.1
- link lidar: mass None -> 0.5; geometry collision cylinder length=0.05 radius=0.1; visual cylinder length=0.05 radius=0.1
- link right_wheel: mass None -> 0.5; geometry collision cylinder length=0.05 radius=0.1; visual cylinder length=0.05 radius=0.1
Joints:
- joint base_caster_wheel_joint: axis 0 1 0 -> (none)
